Commit message: tune parameters

File: roboverse/assets/bullet-objects/drawer/drawer_with_tray_inside.urdf (robot description, URDF)
Before this commit: robot bowl.urdf, 7 links, 6 joints
Links:
- link base: geometry collision box size=.05 1.2 1.4; collision box size=.05 1.2 1.4
- link frame: geometry collision box size=.05 1.3 1.35; collision box size=.05 1.3 1.35
- link tray: geometry collision mesh filename=../tray/tray_textured4_no_color.obj scale=1.1 0.95 3.5; visual mesh filename=../tray/tray_textured4_no_color.obj scale=1.1 0.95 3.5

Commit message: add assets, correct info table clean

File: roboverse/assets/bullet-objects/drawer/drawer_with_tray_inside.urdf (robot description, URDF)
Before this commit: robot bowl.urdf, 7 links, 6 joints
Links:
- link tray: geometry collision mesh filename=../tray/tray_textured4_no_color.obj scale=1.1 0.95 1; visual mesh filename=../tray/tray_textured4_no_color.obj scale=1.1 0.95 3.5
