Commit message: tune parameters

File: roboverse/assets/bullet-objects/drawer/drawer_tableclean.urdf (robot description, URDF)
Before this commit: robot bowl.urdf, 6 links, 5 joints
Links:
- link base: geometry collision box size=.05 1.2 1.31; collision box size=.05 1.2 1.31
- link frame: geometry collision box size=.05 1.3 .6; collision box size=.05 1.3 .6
- link handle_r: geometry collision cylinder length=1.31 radius=0.06; visual cylinder length=1.31 radius=0.06

Commit message: tune parameters

File: roboverse/assets/bullet-objects/drawer/drawer_tableclean.urdf (robot description, URDF)
Before this commit: robot bowl.urdf, 6 links, 5 joints
Links:
- link base: geometry collision box size=.05 1.2 1.4; collision box size=.05 1.2 1.4
- link frame: geometry collision box size=.05 1.3 .6; collision box size=.05 1.3 .6
- link handle_r: geometry collision cylinder length=1.4 radius=0.06; visual cylinder length=1.4 radius=0.06
