Commit message: update office

File: roboverse/assets/room_descriptions/urdf/room_v1.urdf (robot description, URDF)
Before this commit: robot room, 14 links, 13 joints
Links:
- removed link lamp_base
Joints:
- removed joint j_lamp

Commit message: tableclean save

File: roboverse/assets/room_descriptions/urdf/room_v1.urdf (robot description, URDF)
Before this commit: robot room, 13 links, 12 joints
Links:
- added link officedesk, mass 1.0; collision mesh filename=../meshes/obj/wall.obj scale=3 3 3; visual mesh filename=../meshes/obj/officedesk.obj scale=4 4 4
Joints:
- added joint officedesk: type fixed, parent room_base, child officedesk, origin xyz=0 0 0 rpy=0 0 0

Commit message: udpate states

File: roboverse/assets/room_descriptions/urdf/room_v1.urdf (robot description, URDF)
Before this commit: robot room, 12 links, 11 joints
Links:
- removed link deskLamp_base
Joints:
- removed joint j_deskLamp
