Commit message: update office env

File: roboverse/assets/bullet-objects/desktop/desktop.urdf (robot description, URDF)
Before this commit: robot tray, 1 links, 0 joints
Links:
- link tray_base_link: geometry collision mesh filename=cpu.obj scale=0.04 0.04 0.04; visual mesh filename=cpu.obj scale=0.04 0.04 0.04

File: roboverse/assets/bullet-objects/drawer/drawer_tableclean.urdf (robot description, URDF)
Before this commit: robot bowl.urdf, 6 links, 5 joints
Links:
- link base: geometry collision box size=.05 1.2 1.4; collision box size=.05 1.2 1.4
Joints:
- joint handle_plate_far_joint: origin xyz=-0.65 -0.7 0.03 rpy=0 0 0 -> xyz=-0.65 -0.83 0.03 rpy=0 0 0
- joint handle_plate_near_joint: origin xyz=0.65 -0.7 0.03 rpy=0 0 0 -> xyz=0.65 -0.83 0.03 rpy=0 0 0
- joint handle_r_joint: origin xyz=0 -1.1 0.03 rpy=0 0 0 -> xyz=0 -1.2 0.03 rpy=0 0 0

File: roboverse/assets/bullet-objects/monitor/monitor.urdf (robot description, URDF)
Before this commit: robot tray, 1 links, 0 joints
Links:
- link tray_base_link: geometry collision mesh filename=monitor_v1.obj scale=0.65 0.65 0.65; visual mesh filename=monitor_v1.obj scale=0.65 0.65 0.65

File: roboverse/assets/bullet-objects/officedesk/desk.urdf (robot description, URDF)
Before this commit: robot tray, 1 links, 0 joints
Links:
- link tray_base_link: geometry collision box size=1.2 .05 1.4; visual mesh filename=officedesk.obj scale=1 1 1

File: roboverse/assets/room_descriptions/urdf/room_v1.urdf (robot description, URDF)
Before this commit: robot room, 14 links, 13 joints
Links:
- removed link officedesk
- removed link trashcan
- link clock: geometry collision mesh filename=../meshes/obj/clock.obj scale=0.45 0.45 0.5; visual mesh filename=../meshes/obj/clock.obj scale=0.45 0.45 0.5
- link room_base: geometry visual box size=0.001 0.001 0.001
Joints:
- removed joint officedesk
- removed joint trashcan

Commit message: clean up

File: roboverse/assets/bullet-objects/desktop/desktop.urdf (robot description, URDF)
Before this commit: robot tray, 1 links, 0 joints
Links:
- removed link tray_base_link
- added link desktop_base_link, mass 0; collision mesh filename=cpu.obj scale=0.04 0.04 0.04; visual mesh filename=cpu.obj scale=0.04 0.04 0.04

File: roboverse/assets/bullet-objects/eraser/eraser.urdf (robot description, URDF)
Before this commit: robot tray, 1 links, 0 joints
Links:
- removed link tray_base_link
- added link eraser_base_link, mass 0.2; collision mesh filename=eraser.obj scale=0.005 0.01 0.005; visual mesh filename=eraser.obj scale=0.005 0.01 0.005

File: roboverse/assets/bullet-objects/laptop/laptop.urdf (robot description, URDF)
Before this commit: robot tray, 1 links, 0 joints
Links:
- removed link tray_base_link
- added link laptop_base_link, mass 0; collision mesh filename=laptop.obj scale=0.5 0.5 0.5; visual mesh filename=laptop.obj scale=0.5 0.5 0.5

File: roboverse/assets/bullet-objects/monitor/monitor.urdf (robot description, URDF)
Before this commit: robot tray, 1 links, 0 joints
Links:
- removed link tray_base_link
- added link monitor_base_link, mass 0; collision mesh filename=monitor.obj scale=0.65 0.65 0.65; visual mesh filename=monitor.obj scale=0.65 0.65 0.65

File: roboverse/assets/room_descriptions/urdf/room.urdf (robot description, URDF)
Before this commit: robot room, 19 links, 18 joints
Links:
- removed link armchair_base
- removed link beer_base
- removed link chair_base
- removed link commode_base
- removed link deskLamp_base
- removed link desk_base
- removed link lamp_base
- removed link pc_base
- removed link stuff_base
- removed link table_base
- added link books_2_base, mass 0; collision mesh filename=../meshes/obj/books.obj scale=0.012 0.012 0.012; visual mesh filename=../meshes/obj/books.obj scale=0.012 0.012 0.012
- added link clock, mass 0; collision mesh filename=../meshes/obj/clock.obj scale=0.45 0.45 0.5; visual mesh filename=../meshes/obj/clock.obj scale=0.45 0.45 0.5
- link books_base: mass None -> 0; geometry collision mesh filename=../meshes/obj/books.obj scale=0.012 0.012 0.012; visual mesh filename=../meshes/obj/books.obj scale=0.012 0.012 0.012
- link l_box_shelf_1: geometry collision box size=0.2 0.8 0.04; visual box size=0.2 0.8 0.04
- link l_box_shelf_2: geometry collision box size=0.2 0.8 0.04; visual box size=0.2 0.8 0.04
- link l_box_shelf_3: geometry collision box size=0.2 0.8 0.04; visual box size=0.2 0.8 0.04
- link l_box_shelf_4: geometry collision box size=0.2 0.8 0.04; visual box size=0.2 0.8 0.04
- link l_carpet: mass None -> 0; geometry collision mesh filename=../meshes/obj/carpet.obj; visual mesh filename=../meshes/obj/carpet.obj
- link l_carpet_wall_one: geometry collision mesh filename=../meshes/obj/wall.obj scale=1 1 1.5; visual mesh filename=../meshes/obj/wall.obj scale=1 1 1.5
- link l_carpet_wall_two: geometry collision mesh filename=../meshes/obj/wall.obj scale=1 1 1.5; visual mesh filename=../meshes/obj/wall.obj scale=1 1 1.5
- link room_base: mass None -> 0; geometry visual box size=0.001 0.001 0.001
Joints:
- removed joint j_armchair
- removed joint j_beer
- removed joint j_chair
- removed joint j_commode
- removed joint j_desk
- removed joint j_deskLamp
- removed joint j_lamp
- removed joint j_pc
- removed joint j_stuff
- removed joint j_table
- added joint clock: type fixed, parent room_base, child clock, origin xyz=0 0 0 rpy=0 0 0
- added joint j_books_2: type fixed, parent room_base, child books_2_base, origin xyz=0 0 0 rpy=0 0 0
